File: vga_test.kicad_sch (KiCad schematic)
At the start: 34 parts, among them J1 DE15_Receptacle_HighDensity_M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, J10 Conn_01x04, J11 Conn_02x02_Odd_Even, J12 Conn_01x08, J2 Conn_02x03_Counter_Clockwise, J3 Conn_02x02_Odd_Even, J4 Conn_01x03, J5 Conn_01x04, J6 Conn_01x04, J7 Conn_01x04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

Commit message: added more text
Parts:
- J1: footprint Library:DSUB-15-L77HDE15SD1CH4F -> vga:DSUB-15-L77HDE15SD1CH4F
Changed lines of the file:
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@@
 			)
 		)
-		(property "Footprint" "Library:DSUB-15-L77HDE15SD1CH4F"
+		(property "Footprint" "vga:DSUB-15-L77HDE15SD1CH4F"
 			(at 13.97 34.29 0)
 			(effects
